File: Schematics/HRV_Control.brd (EAGLE design)
At the start: 68.2 x 66 mm, 32 parts, among them IC1 5v

Commit message: Misc. enhancements
- Revised algorithms for fresh air and dehumidification for improved
efficiency.
- Added ClearEeprom function initiatated by sending code 5 from to
microprocessor.
- Revised circuit board to fix errors with voltage regulator pinout and
resistor sizes.
Parts:
- C1: device resistor:C025-024X044 -> capacitor-wima:C5B3
- IC1: value 5v -> (none); device v-reg:79XXS -> v-reg:78XXL
- R1, R2, R3, R4, R5, R6, R7: device resistor:0204/5 -> resistor:0204/7
- moved C1 16.6 mm to (14.0, 5.08)
- moved IC1 4.58 mm to (7.62, 16.5)
- moved R1 1.27 mm to (53.3, 22.9)
- moved R2 1.27 mm to (47.0, 22.9)
- moved R3 1.27 mm to (40.6, 22.9)
- moved R5 1.27 mm to (15.2, 27.9)
Routing:
- net VCC: track 168.1 -> 189.1 mm
- net N$18: track 56.3 -> 42.6 mm
- net N$1: track 59.4 -> 46.6 mm
- net N$3: track 42.1 -> 34.6 mm
- net STX: track 46.0 -> 51.0 mm
- net SRX: track 25.8 -> 30.4 mm
- net N$14: track 37.7 -> 42.0 mm
- net N$13: track 34.8 -> 37.3 mm
- net N$7: track 29.1 -> 30.1 mm
- net N$8: track 33.2 -> 34.2 mm, vias 1 -> 0
- net N$12: track 45.6 -> 46.5 mm
- net N$17: track 44.7 -> 45.5 mm
